File: hardware/main board/MotorControl.kicad_sch (KiCad schematic)
At the start: 5 parts, among them IC2 DRV8212PDSGR, IC6 SN74LVC1G18DBVRG4

Commit message: done
Parts:
- renumbered C14 to C18, IC6 to IC7
Changed lines of the file:
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@@
 		(dnp no)
 		(fields_autoplaced yes)
-		(property "Reference" "IC6"
+		(property "Reference" "IC7"
 			(at 162.56 81.28 0)
 			(effects
@@
 		(on_board yes)
 		(dnp no)
-		(property "Reference" "#PWR06"
+		(property "Reference" "#PWR017"
 			(at 149.86 101.6 0)
 			(effects
@@
 		(on_board yes)
 		(dnp no)
-		(property "Reference" "C14"
+		(property "Reference" "C18"
 			(at 90.17 76.2 90)
 			(effects
@@
 		(dnp no)
 		(fields_autoplaced yes)
-		(property "Reference" "#PWR06"
+		(property "Reference" "#PWR017"
 			(at 128.27 81.28 0)
 			(effects

Commit message: final
Other:
- company: (none) -> Made by: Piotr Lesicki
- title: (none) -> Mirco Mouse
Changed lines of the file:
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@@
 	(generator_version "8.0")
 	(paper "A4")
+	(title_block
+		(title "Mirco Mouse")
+		(date "2025-01-02")
+		(rev "1.0")
+		(company "Made by: Piotr Lesicki")
+	)
 	(junction
 		(at 129.54 81.28)
@@
 		(dnp no)
 		(property "Reference" "C19"
-			(at 143.51 105.41 0)
-			(effects
-				(font
-					(size 1.27 1.27)
-				)
+			(at 146.05 105.6386 0)
+			(effects
+				(font
+					(size 1.27 1.27)
+				)
+				(justify left)
 			)
 		)
 		(property "Value" "100nF"
-			(at 143.51 107.7214 0)
-			(effects
-				(font
-					(size 1.27 1.27)
-				)
+			(at 146.05 107.95 0)
+			(effects
+				(font
+					(size 1.27 1.27)
+				)
+				(justify left)
 			)
 		)
@@
 		(dnp no)
 		(property "Reference" "C19"
-			(at 134.62 77.47 0)
-			(effects
-				(font
-					(size 1.27 1.27)
-				)
+			(at 132.08 74.7014 0)
+			(effects
+				(font
+					(size 1.27 1.27)
+				)
+				(justify left)
 			)
 		)
 		(property "Value" "100nF"
-			(at 134.62 75.1586 0)
-			(effects
-				(font
-					(size 1.27 1.27)
-				)
+			(at 132.08 77.47 0)
+			(effects
+				(font
+					(size 1.27 1.27)
+				)
+				(justify left)
 			)
 		)
@@
 		(dnp no)
 		(property "Reference" "C18"
-			(at 90.17 76.2 90)
-			(effects
-				(font
-					(size 1.27 1.27)
-				)
+			(at 93.98 74.93 0)
+			(effects
+				(font
+					(size 1.27 1.27)
+				)
+				(justify left)
 			)
 		)
 		(property "Value" "4.7uF"
-			(at 92.71 76.2 90)
-			(effects
-				(font
-					(size 1.27 1.27)
-				)
-			)
-		)
+			(at 93.98 77.47 0)
+			(effects
+				(font
+					(size 1.27 1.27)
+				)
+				(justify left)
+			)
+		)
